File: eagle/metroid/untitled.sch (EAGLE design)
At the start: 4 parts, among them IC1 MEGA48/88/168-AU, U1 AT45DB321D-S

Commit message: before adding humidity
Parts:
- added C1: 1uF, ng:UNPOLARIZED_CAPACITOR1206
- added C2, C3, C4, C5, C6: .1uF, ng:UNPOLARIZED_CAPACITOR1206
- added IC4: MIC5219BM5, metrify:MIC5219BM5
- added PWR: (no value), con-lstb:MA03-1
- added Q1: (no value), crystal:CRYSTALTC26H
- added S1: (no value), fab:6MM_SWITCH6MM_SWITCH
- added SV1: (no value), con-lstb:MA04-2
- added SV2: (no value), con-lstb:MA08-1
- added U$1: BS-7BATTERYCLIP, metrify:BS-7BATTERYCLIP
- added U$2: DS18S20, metrify:DS18S20
Connections:
- net N$1 renamed PORTC
- removed net +5V: WRL-00691.1
- new net N$1: C6.2, IC1.AREF
- new net N$10: IC1.PC4(ADC4/SDA/PCINT12), SV2.5
- new net N$11: IC1.PC5(ADC5/SCL/PCINT13), SV2.6
- new net N$12: IC1.ADC6, SV2.7
- new net N$13: IC1.ADC7, SV2.8
- new net N$14: IC4.IN, IC4.SD, PWR.3
- new net N$3: IC1.PB6(XTAL1/TOSC1/PCINT6), Q1.2
- new net N$4: IC1.PB7(XTAL2/TOSC2/PCINT7), Q1.1
- new net N$5: IC1.PD4(T0/XCK/PCINT20), U$2.DQ
- new net N$6: IC1.PC0(ADC0/PCINT8), S1.P, S1.P1, SV2.1
- new net N$7: IC1.PC1(ADC1/PCINT9), SV2.2
- new net N$8: IC1.PC2(ADC2/PCINT10), SV2.3
- new net N$9: IC1.PC3(ADC3/PCINT11), SV2.4
- net +3V3: now also C1.2, C2.2, C3.2, C4.2, C5.2, IC1.AVCC, IC4.OUT, PWR.2, SV1.7, U$1.POS, U$2.VCC, WRL-00691.1
- net GND: now also C1.1, C2.1, C3.1, C4.1, C5.1, C6.1, IC1.AGND, IC4.GND, PWR.1, S1.S, S1.S1, SV1.8, U$1.NEG, U$2.GND
- net MISO: now also SV1.2
- net MOSI: now also SV1.3
- net RFCEN: now also SV1.6
- net RFIRQ: now also SV1.1
- net RFSPICS: now also SV1.5
- net SCK: now also SV1.4

Commit message: board routed. eagle 6. 6 mil traces, qfp atmega+battery+labpowerheaders+headers>sparkfunnordic or mdfly+pads for 1206 sensors, humidity, phototransistor+isp+pushbutton
Parts:
- removed C2, C5, C6: .1uF, ng:UNPOLARIZED_CAPACITOR1206
- added CSENSE: (no value), rcl:CPOL-USE5-8.5
- added EXTPWR: (no value), rcl:R-US_M0805
- added PD: (no value), ng:PHOTOTRANSISTOR5MM
- added RBRIDGE, RCAP, RPD: (no value), ng:RESISTOR1206
- added RSENSE: (no value), rcl:R-US_0207/7
- JP1: value AVR-ISP-6VERT -> AVR-ISP
- SV1: value (none) -> RF-IS2411
- SV2: value (none) -> ADC; device con-lstb:MA08-1 -> con-lstb:MA10-1
Connections:
- net N$5 renamed 1WIRE
- removed net N$1: C6.2, IC1.AREF
- removed net N$7: IC1.PC1(ADC1/PCINT9), SV2.2
- new net AUXSENSE: IC1.PD3(INT1/OC2B/PCINT19), RBRIDGE.2, RCAP.2, RPD.2
- new net HUMIDITY: CSENSE.+, IC1.PB1(OC1A/PCINT1), RCAP.1
- new net N$15: IC1.ADC6, SV2.3
- new net N$5: EXTPWR.1, IC4.OUT
- new net PHOTODIODE: IC1.PB0(ICP1/CLKO/PCINT0), PD.C, RPD.1
- new net RBRIDGE: IC1.PB2(SS/OC1B/PCINT2), RBRIDGE.1, RSENSE.2
- net +3V3: now also EXTPWR.2, PWR.3, SV2.1; no longer C2.2, C5.2, IC4.OUT, PWR.2
- net GND: now also CSENSE.-, PD.E, RSENSE.1, SV2.2; no longer C2.1, C5.1, C6.1
- net N$10: now also IC1.PC3(ADC3/PCINT11), SV2.8; no longer IC1.PC4(ADC4/SDA/PCINT12), SV2.5
- net N$11: now also IC1.PC4(ADC4/SDA/PCINT12), SV2.9; no longer IC1.PC5(ADC5/SCL/PCINT13), SV2.6
- net N$12: now also IC1.PC5(ADC5/SCL/PCINT13), SV2.10; no longer IC1.ADC6, SV2.7
- net N$13: now also SV2.4; no longer SV2.8
- net N$14: now also PWR.2; no longer PWR.3
- net N$6: now also SV2.5; no longer SV2.1
- net N$8: now also IC1.PC1(ADC1/PCINT9), SV2.6; no longer IC1.PC2(ADC2/PCINT10), SV2.3
- net N$9: now also IC1.PC2(ADC2/PCINT10), SV2.7; no longer IC1.PC3(ADC3/PCINT11), SV2.4
Other:
- moved on the sheet: C1, IC4, PWR, S1
